File: hardware/YamuraHub_T41/YamuraHub_T41.kicad_sch (KiCad schematic)
At the start: 29 parts, among them J1 12V in, J2 CAN H/L (from A3), J3 DB9 male - CAN bus, J4 Display (MSP4030/4031 14-pin), J5 I2C (Wire2) / GPS, J6 Panel buttons, J7 Panel LEDs, SW1 SELECT, SW2 UP, SW3 DOWN, U1 R-78E5.0-1.0

Commit message: Hub carrier board rev B: display on front, parts on back, two DB9s
- 122 x 68 mm board: the 4" display (MSP4030/4031) plugs into J4 on the
  front, long side along the board, on M3 standoffs at its own holes
  (H5-H8); every other part is on the back; M3 holes at the corners.
- Second DB9 (J8) in parallel with J3 so the CAN bus can pass through
  the hub. Waveshare terminator must come off if both are used.
- Buttons and LEDs are panel-mounted: SW1-3 and D2/D3 removed, J6/J7
  headers kept (R1/R2 still on board).
- build_pcb.py flips side "B" parts to the back with mirrored back-side
  silkscreen and draws the display outline on the front.
- route.py rips up and retries with failed nets first; pad stubs only
  from real track endpoints.
- Fab outputs, BOM, renders and README regenerated for rev B.

ERC clean; DRC with schematic parity: 0 unconnected, 0 mismatches,
no courtyard/clearance errors (two starved-thermal warnings only).

Co-Authored-By: Claude Opus 5.5 <noreply@anthropic.com>
Parts:
- removed D2: Red (REC), LED_THT:LED_D5.0mm, symbol Device:LED
- removed D3: Green (GPS), LED_THT:LED_D5.0mm, symbol Device:LED
- removed J6: Panel buttons, Connector_PinHeader_2.54mm:PinHeader_1x04_P2.54mm_Vertical, symbol Connector_Generic:Conn_01x04
- removed SW1: SELECT, Button_Switch_THT:SW_PUSH_6mm, symbol Switch:SW_Push
- removed SW3: DOWN, Button_Switch_THT:SW_PUSH_6mm, symbol Switch:SW_Push
- added H1, H2, H3, H4: M3 (board), MountingHole:MountingHole_3.2mm_M3, symbol Mechanical:MountingHole
- added J1: 12V in, TerminalBlock_Phoenix:TerminalBlock_Phoenix_MKDS-1,5-2-5.08_1x02_P5.08mm_Horizontal, symbol Connector:Screw_Terminal_01x02
- H5: renamed from H1; value M3 -> M3 (display)
- H6: renamed from H2; value M3 -> M3 (display)
- H7: renamed from H3; value M3 -> M3 (display)
- H8: renamed from H4; value M3 -> M3 (display)
- J3: value DB9 male - CAN bus -> DB9 male - CAN bus 1
- J4: value Display (MSP4030/4031 14-pin) -> Display socket (MSP4030/4031 14-pin); footprint Connector_PinHeader_2.54mm:PinHeader_1x14_P2.54mm_Vertical -> Connector_PinSocket_2.54mm:PinSocket_1x14_P2.54mm_Vertical
- J6: renamed from SW2; value UP -> Panel buttons; footprint Button_Switch_THT:SW_PUSH_6mm -> Connector_PinHeader_2.54mm:PinHeader_1x04_P2.54mm_Vertical; symbol Switch:SW_Push -> Connector_Generic:Conn_01x04
- J8: renamed from J1; value 12V in -> DB9 male - CAN bus 2; footprint TerminalBlock_Phoenix:TerminalBlock_Phoenix_MKDS-1,5-2-5.08_1x02_P5.08mm_Horizontal -> Connector_Dsub:DSUB-9_Pins_Horizontal_P2.77x2.84mm_EdgePinOffset7.70mm_Housed_MountingHolesOffset9.12mm; symbol Connector:Screw_Terminal_01x02 -> Connector:DE9_Pins_MountingHoles
Connections:
- net +12V_BUS: now also J8.9
- net +12V_IN: now also J1.1 (Pin_1); no longer J8.1 (Pin_1)
- net BTN_DOWN: now also J6.3 (Pin_3)
- net BTN_SELECT: now also J6.1 (Pin_1)
- net BTN_UP: now also J6.2 (Pin_2); no longer J6.1
- net CANH: now also J8.7
- net CANL: now also J8.2
- net GND: now also J6.4 (Pin_4), J8.3, J8.6, J8.SH (PAD), J1.2 (Pin_2); no longer J6.2, J8.2 (Pin_2)
- no-connect marks 37 -> 41
Other:
- note added: "JP1 open by default: ST7796 SDO does not tri-state and would contend with the AirLift on MISO. A3 (Waveshare) has a fixed 120R terminator: remove it if both DB9s are used (hub mid-bus)."
- note removed: "JP1 open by default: ST7796 SDO does not tri-state and would contend with the AirLift on MISO. A3 (Waveshare) includes a 120R terminator - hub is the bus end."
- moved on the sheet: H5, H6, H7, H8, J3
